File: pcb/TI74_RAM.sch (EAGLE design)
At the start: 10 parts, among them IC1 JEDEC_32KB_SRAM, X1 TI74_CONNREG

Commit message: Add in A14 address line
Parts:
- added GOLD_ORB_SM1: Open Source Hardware, oshw:OSHWLOGOLOGO5MM
- C1: value 100 -> 100n; device resistor:C-USC1206 -> resistor:C-USC0603
- C2: value 1 -> 1n
Connections:
- net A1: now also IC1A.A7; no longer IC1A.A6
- net A10: now also IC1A.A4; no longer IC1A.A3
- net A14: now also IC1A.A9
- net A2: now also IC1A.A6; no longer IC1A.A5
- net A4: now also IC1A.A10; no longer IC1A.A11
- net A5: now also IC1A.A11; no longer IC1A.A9
- net A6: now also IC1A.A5; no longer IC1A.A4
- net A7: now also IC1A.A3; no longer IC1A.A10
- net A8: now also IC1A.A14; no longer IC1A.A12
- net A9: now also IC1A.A12; no longer IC1A.A7
- net GND: no longer IC1A.A14
- net N$2: now also D2.A; no longer D1.A
- net N$3: now also D1.A; no longer D2.A
Other:
- moved on the sheet: D1, D2
